File: 8x18650.kicad_pcb (KiCad board)
At the start: 2 copper layers, 176 x 78 mm, 9 parts, among them J1 B3B-XH-A, J8 BH-18650-PC8, J9 BH-18650-PC8

Commit message: Updated license information
Other:
- board text added: "Copyright Taiyo Rawle 2025 Released under CERN OHL 2.0-S"
Changed lines of the file:
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@@
 		(tags "connector JST XH vertical boss")
 		(property "Reference" "J1"
-			(at -4 0 360)
+			(at -4 0 0)
 			(layer "F.SilkS")
 			(effects
@@
 		(layer "Edge.Cuts")
 	)
+	(gr_text "Copyright Taiyo Rawle 2025\nReleased under CERN OHL 2.0-S"
+		(at 148 108 0)
+		(layer "B.Cu")
+		(effects
+			(font
+				(size 1.5 1.5)
+				(thickness 0.25)
+				(bold yes)
+			)
+			(justify mirror)
+		)
+	)
 	(gr_text "Affix foam here"

Commit message: Updated license infomration.
Other:
- board text added: "HAOS REDRO PN: 0000.011B by Taiyo Rawle is marked with CC0 1.0"
- board text removed: "Copyright Taiyo Rawle 2025 Released under CERN OHL 2.0-S"
Changed lines of the file:
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@@
 	)
 	(paper "A4")
+	(title_block
+		(comment 3 "HAOS REDRO PN: 0000.011B by Taiyo Rawle is marked with CC0 1.0 ")
+	)
 	(layers
 		(0 "F.Cu" signal)
@@
 		(layer "Edge.Cuts")
 	)
-	(gr_text "Copyright Taiyo Rawle 2025\nReleased under CERN OHL 2.0-S"
+	(gr_text "HAOS REDRO PN: 0000.011B by\nTaiyo Rawle is marked with CC0 1.0 "
 		(at 148 108 0)
 		(layer "B.Cu")
