File: 8x18650.kicad_sch (KiCad schematic)
At the start: 9 parts, among them J1 B3B-XH-A, J8 BH-18650-PC8, J9 BH-18650-PC8

Commit message: Updated license infomration.
Other:
- company: HAOS REDRO PN: 0000 0001 -> HAOS REDRO PN: 0000 011B
Changed lines of the file:
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@@
 	(title_block
 		(title "Stackable holder for eight 18650 cells")
-		(date "2019-01-30")
+		(date "2025-01-26")
 		(rev "1.0")
-		(company "HAOS REDRO PN: 0000 0001")
+		(company "HAOS REDRO PN: 0000 011B")
 		(comment 1 "https://www.haosredro.com")
-		(comment 2 "Licensed under CERN OHL 2.0-S")
+		(comment 2 "HAOS REDRO PN: 0000.011B by Taiyo Rawle is marked with CC0 1.0 ")
 	)
 	(junction
